Commit message: Added simple pendulum model and fixed pendulum gazebo compatible model, finally worksgit add .git add .

File: simple_pendulum/simple_pedulum_description/urdf/simple_pedulum.xacro (robot description, xacro)
@@ -44,5 +44,5 @@
   </collision>
 </link>
-<joint name="Ball2" type="Ball">
+<joint name="Ball2" type="continuous">
   <origin xyz="0.0125 0.012 0.175" rpy="0 0 0"/>
   <parent link="base_link"/>
